Commit message: add v1 mesh back
Signed-off-by: Mabel Zhang <mabel@openrobotics.org>

File: cora_description/urdf/cora_v1.urdf.xacro (robot description, xacro)
@@ -10,10 +10,10 @@
     <visual>
       <geometry>
-        <mesh filename="package://cora_description/models/base/meshes/base.dae"/>
+        <mesh filename="package://cora_description/models/base/meshes/base_v1.dae"/>
       </geometry>
     </visual>
     <collision name="collision">
       <geometry>
-        <box size="12.21 3.58 2.84" />
+        <box size="12.21 3.58 3.53" />
       </geometry>
     </collision>
@@ -23,6 +23,6 @@
       <mass value="42.935"/>
       <inertia ixx="55.373356" ixy="0.245103" ixz="-21.590300"
-                                iyy="341.188965" iyz="0.053122"
-                                                 izz="367.665375"/>
+                               iyy="341.188965" iyz="0.053122"
+                                                izz="367.665375"/>
     </inertial>
   </link>
