Commit message: fix engine inertia
Signed-off-by: Mabel Zhang <mabel@openrobotics.org>

File: cora_description/urdf/thrusters.xacro (robot description, xacro)
@@ -5,5 +5,5 @@
     <inertial>
       <mass value="0.1"/>
-      <inertia ixx="0.889245" ixy="0.0" ixz="0.0" iyy="0.911125" iyz="0.0" izz="0.078125"/>
+      <inertia ixx="0.00889245" ixy="0.0" ixz="0.0" iyy="0.00911125" iyz="0.0" izz="0.00078125"/>
     </inertial>
   </link>
@@ -40,5 +40,5 @@
     <inertial>
       <mass value="0.1"/>
-      <inertia ixx="0.889245" ixy="0.0" ixz="0.0" iyy="0.911125" iyz="0.0" izz="0.078125"/>
+      <inertia ixx="0.00889245" ixy="0.0" ixz="0.0" iyy="0.00911125" iyz="0.0" izz="0.00078125"/>
     </inertial>
   </link>
