Commit message: move to cora_description package
Signed-off-by: Mabel Zhang <mabel@openrobotics.org>

File: cora_description/urdf/cora_dynamics_plugin.xacro (robot description, xacro)
@@ -12,7 +12,7 @@
         <xDotU>0</xDotU>
         <yDotV>26000</yDotV>
-	<zDotW>31000</zDotW>
-	<kDotP>0.0</kDotP>
-	<mDotQ>0.0</mDotQ>
+        <zDotW>31000</zDotW>
+        <kDotP>0.0</kDotP>
+        <mDotQ>0.0</mDotQ>
         <nDotR>0.0</nDotR>
         <!-- Linear and quadratic drag -->
@@ -22,9 +22,9 @@
         <yVV>2600</yVV>
         <zW>50000.0</zW>
-	<zWW>0.0</zWW>
+        <zWW>0.0</zWW>
         <kP>50000.0</kP>
-	<kPP>5000.0</kPP>
+        <kPP>5000.0</kPP>
         <mQ>500000.0</mQ>
-	<mQQ>5000.0</mQQ>
+        <mQQ>5000.0</mQQ>
         <nR>400000.0</nR>
         <nRR>0.0</nRR>

File: cora_description/urdf/cora_thruster_config.xacro (robot description, xacro)
@@ -1,5 +1,5 @@
 <?xml version="1.0"?>
 <plugin xmlns:xacro="http://ros.org/wiki/xacro">
-  <xacro:macro  name="cora_gazebo_thruster_config" params="name">
+  <xacro:macro  name="cora_thruster_config" params="name">
     <thruster>
       <!-- Required Parameters -->

File: cora_description/urdf/macros.xacro (robot description, xacro)
@@ -13,4 +13,4 @@
   <xacro:include filename="$(find wamv_gazebo)/urdf/sensors/wamv_pinger.xacro" />
   <!-- Include dynamics macros -->
-  <xacro:include filename="$(find cora_gazebo)/urdf/cora_gazebo_dynamics_plugin.xacro" />
+  <xacro:include filename="$(find cora_description)/urdf/cora_dynamics_plugin.xacro" />
 </robot>

File: cora_description/urdf/thrusters.xacro (robot description, xacro)
@@ -75,8 +75,8 @@
       <cmdTimeout>1.0</cmdTimeout>
       <robotNamespace>${namespace}</robotNamespace>
-      <xacro:include filename="$(find cora_gazebo)/urdf/cora_gazebo_thruster_config.xacro" />
+      <xacro:include filename="$(find cora_description)/urdf/cora_thruster_config.xacro" />
       <!-- Angle must be disabled for VORC -->
-      <xacro:cora_gazebo_thruster_config name="left" />
-      <xacro:cora_gazebo_thruster_config name="right" />
+      <xacro:cora_thruster_config name="left" />
+      <xacro:cora_thruster_config name="right" />
     </plugin>
   </gazebo>
