Commit message: thrusters and control
Signed-off-by: Mabel Zhang <mabel@openrobotics.org>

File: cora_description/urdf/cora.xacro (robot description, xacro)
@@ -7,3 +7,11 @@
   <!-- Robot mesh -->
   <xacro:include filename="$(find cora_description)/urdf/cora.urdf.xacro" />
+  <!-- Note: this is only used for some sensors that do not correctly use the
+  robotNamespace parameter -->
+  <xacro:arg name="namespace" default="cora"/>
+  <xacro:property name="namespace" value="$(arg namespace)" scope="global" />
+  <!-- Thrusters -->
+  <xacro:arg name="thruster_namespace" default="thrusters/"/>
+  <xacro:property name="thruster_namespace" value="$(arg thruster_namespace)" scope="global" />
+  <xacro:include filename="$(find cora_description)/urdf/thrusters.xacro" />
 </robot>

Commit message: Adding sensors to CoRa (#2)
* Adding sensors with preliminary location.

Signed-off-by: Carlos Agüero <caguero@openrobotics.org>

* Install config dir.

Signed-off-by: Carlos Agüero <caguero@openrobotics.org>

File: cora_description/urdf/cora.xacro (robot description, xacro)
@@ -15,3 +15,16 @@
   <xacro:property name="thruster_namespace" value="$(arg thruster_namespace)" scope="global" />
   <xacro:include filename="$(find cora_description)/urdf/thrusters.xacro" />
+  <!-- Sensors -->
+  <xacro:arg name="camera_namespace" default="cameras/"/>
+  <xacro:arg name="sensor_namespace" default="sensors/"/>
+  <xacro:arg name="pinger_namespace" default="pingers/"/>
+  <xacro:property name="camera_namespace" value="$(arg camera_namespace)" scope="global" />
+  <xacro:property name="sensor_namespace" value="$(arg sensor_namespace)" scope="global" />
+  <xacro:property name="pinger_namespace" value="$(arg pinger_namespace)" scope="global" />
+  <xacro:wamv_camera name="front_left_camera"  y="0.1"  x="3.75" z="1.6" P="${radians(15)}" />
+  <xacro:wamv_camera name="front_right_camera" y="-0.1" x="3.75" z="1.6" P="${radians(15)}" />
+  <xacro:lidar name="front_lidar" type="16_beam" x="3.75" z="1.8" />
+  <xacro:wamv_gps name="gps" x="-0.4" z="1.4" />
+  <xacro:wamv_imu name="imu" y="-0.2" />
+  <xacro:wamv_pinger name="pinger" position="1.0 0 -1.0" />
 </robot>

Commit message: lock boat; lift sensor positions higher; move buoys farther ahead
Signed-off-by: Mabel Zhang <mabel@openrobotics.org>

File: cora_description/urdf/cora.xacro (robot description, xacro)
@@ -1,4 +1,5 @@
 <?xml version="1.0"?>
 <robot xmlns:xacro="http://ros.org/wiki/xacro" name="cora">
+  <xacro:arg name="locked" default="false" />
   <!-- Include macros for dynamics plugins -->
   <xacro:include filename="$(find cora_description)/urdf/macros.xacro" />
@@ -15,4 +16,31 @@
   <xacro:property name="thruster_namespace" value="$(arg thruster_namespace)" scope="global" />
   <xacro:include filename="$(find cora_description)/urdf/thrusters.xacro" />
+  <!-- Decide if we lock the robot to the world -->
+  <xacro:if value="$(arg locked)">
+    <gazebo>
+      <link name="cora_external_link"/>
+      <joint name="cora_external_pivot_joint" type="universal">
+        <parent>cora::base_link</parent>
+        <child>cora_external_link</child>
+        <axis>
+          <xyz>1 0 0</xyz>
+        </axis>
+        <axis2>
+          <xyz>0 1 0</xyz>
+        </axis2>
+      </joint>
+      <joint name="cora_external_riser" type="prismatic">
+        <parent>world</parent>
+        <child>cora_external_link</child>
+        <axis>
+          <limit>
+            <lower>-3</lower>
+            <upper>3</upper>
+          </limit>
+          <xyz>0 0 1</xyz>
+        </axis>
+      </joint>
+    </gazebo>
+  </xacro:if>
   <!-- Sensors -->
   <xacro:arg name="camera_namespace" default="cameras/"/>
@@ -22,9 +50,9 @@
   <xacro:property name="sensor_namespace" value="$(arg sensor_namespace)" scope="global" />
   <xacro:property name="pinger_namespace" value="$(arg pinger_namespace)" scope="global" />
-  <xacro:wamv_camera name="front_left_camera"  y="0.1"  x="3.75" z="1.6" P="${radians(15)}" />
-  <xacro:wamv_camera name="front_right_camera" y="-0.1" x="3.75" z="1.6" P="${radians(15)}" />
-  <xacro:lidar name="front_lidar" type="16_beam" x="3.75" z="1.8" />
-  <xacro:wamv_gps name="gps" x="-0.4" z="1.4" />
-  <xacro:wamv_imu name="imu" y="-0.2" />
+  <xacro:wamv_camera name="front_left_camera"  y="0.1"  x="3.75" z="2.6" P="${radians(15)}" />
+  <xacro:wamv_camera name="front_right_camera" y="-0.1" x="3.75" z="2.6" P="${radians(15)}" />
+  <xacro:lidar name="front_lidar" type="16_beam" x="3.75" z="2.8" />
+  <xacro:wamv_gps name="gps" x="-0.4" z="2.4" />
+  <xacro:wamv_imu name="imu" y="-0.2" z="1"/>
   <xacro:wamv_pinger name="pinger" frameId="cora/pinger" />
 </robot>

File: vorc_gazebo/worlds/perception_task.world.xacro (robot description, xacro)
@@ -44,5 +44,5 @@
           <type>surmark950410</type>
           <name>red_0</name>
-          <pose>8 0 1 0 0 0</pose>
+          <pose>15 0 1 0 0 0</pose>
         </object>
         <object>
@@ -50,5 +50,5 @@
           <type>surmark950400</type>
           <name>green_0</name>
-          <pose>8 2 1 0 0 0</pose>
+          <pose>15 2 1 0 0 0</pose>
         </object>
         <object>
@@ -56,5 +56,5 @@
           <type>black_totem</type>
           <name>black_0</name>
-          <pose>8 -2 1 0 0 0</pose>
+          <pose>15 -2 1 0 0 0</pose>
         </object>
       </object_sequence>
