Commit message: fix inertia, model authors, add dynamic plugin, etc
Signed-off-by: Mabel Zhang <mabel@openrobotics.org>

File: cora_description/urdf/cora.urdf.xacro (robot description, xacro)
@@ -6,5 +6,4 @@
     <parent link="base_link"/>
     <child link="dummy_link"/>
-    <!--pose>0 0 0 1.57 0 1.57</pose-->
   </joint>
   <link name="dummy_link">
@@ -15,15 +14,16 @@
     </visual>
     <collision name="collision">
+      <origin xyz="0 0 0.262063" rpy="0 0 0" />
       <geometry>
-        <box size="3.58 3.53 12.21" />
+        <box size="12.21 3.58 3.53" />
       </geometry>
     </collision>
     <!-- Numbers are from MeshLab -->
     <inertial>
-      <pose>0 0.461760 0.262063</pose>
+      <origin xyz="0.461760 0 0.262063" rpy="0 0 0" />
       <mass value="50.964"/>
-      <inertia ixx="396.178589" ixy="0.0" ixz="0.0"
-                                iyy="418.985809" iyz="-25.942278"
-                                                 izz="71.063889"/>
+      <inertia ixx="71.068199" ixy="0.0" ixz="-25.944702"
+                                iyy="396.183960" iyz="0.0"
+                                                 izz="418.985809"/>
     </inertial>
   </link>

File: cora_description/urdf/cora.xacro (robot description, xacro)
@@ -3,9 +3,10 @@
   <xacro:macro  name="robot_gazebo">
     <!-- Include macros for dynamics plugins -->
-    <!--xacro:include filename="$(find cora_description)/urdf/macros.xacro" /-->
+    <xacro:include filename="$(find cora_description)/urdf/macros.xacro" />
     <!-- Defines the base vehicle -->
     <xacro:include filename="$(find cora_description)/urdf/cora.urdf.xacro" />
     <!-- Attach hydrodynamics plugin -->
-    <xacro:usv_dynamics_gazebo name="cora_dynamics_plugin"/>
+    <xacro:usv_dynamics_gazebo name="cora_dynamics_plugin"
+        width="3.58" length="12.21"/>
   </xacro:macro>
 </robot>

File: vorc_gazebo/worlds/marina.world.xacro (robot description, xacro)
@@ -12,5 +12,5 @@
       <wind_objs>
         <wind_obj>
-          <name>cora_wind</name>
+          <name>cora</name>
           <link_name>base_link</link_name>
           <coeff_vector>0.5 0.5 0.33</coeff_vector>

Commit message: recenter robot model
Signed-off-by: Mabel Zhang <mabel@openrobotics.org>

File: cora_description/urdf/cora.urdf.xacro (robot description, xacro)
@@ -14,5 +14,4 @@
     </visual>
     <collision name="collision">
-      <origin xyz="0 0 0.262063" rpy="0 0 0" />
       <geometry>
         <box size="12.21 3.58 3.53" />

Commit message: new robot mesh without cabin
Signed-off-by: Mabel Zhang <mabel@openrobotics.org>

File: cora_description/urdf/cora.urdf.xacro (robot description, xacro)
@@ -19,14 +19,14 @@
     <collision name="collision">
       <geometry>
-        <box size="12.21 3.58 3.53" />
+        <box size="12.21 3.58 2.84" />
       </geometry>
     </collision>
     <!-- Numbers are from MeshLab -->
     <inertial>
-      <origin xyz="0.461760 0 0.262063" rpy="0 0 0" />
-      <mass value="50.964"/>
-      <inertia ixx="71.068199" ixy="0.0" ixz="-25.944702"
-                                iyy="396.183960" iyz="0.0"
-                                                 izz="418.985809"/>
+      <origin xyz="0.458797 0.002028 0.234834" rpy="0 0 0" />
+      <mass value="42.935"/>
+      <inertia ixx="55.373356" ixy="0.245103" ixz="-21.590300"
+                                iyy="341.188965" iyz="0.053122"
+                                                 izz="367.665375"/>
     </inertial>
   </link>

Commit message: Adding sensors with preliminary location.
Signed-off-by: Carlos Agüero <caguero@openrobotics.org>

File: cora_description/urdf/cora.urdf.xacro (robot description, xacro)
@@ -1,6 +1,31 @@
 <?xml version="1.0"?>
 <robot xmlns:xacro="http://ros.org/wiki/xacro" name="cora">
+  <xacro:arg name="locked" default="false" />
+  <xacro:arg name="ground_truth_enabled" default="false" />
+  <xacro:arg name="thruster_namespace" default="thrusters/"/>
+  <xacro:arg name="camera_namespace" default="cameras/"/>
+  <xacro:arg name="sensor_namespace" default="sensors/"/>
+  <xacro:arg name="pinger_namespace" default="pingers/"/>
+  <!-- Note: this is only used for some sensors that do not correctly use the
+  robotNamespace parameter -->
+  <xacro:arg name="namespace" default="cora"/>
+  <xacro:property name="thruster_namespace" value="$(arg thruster_namespace)" scope="global" />
+  <xacro:property name="camera_namespace" value="$(arg camera_namespace)" scope="global" />
+  <xacro:property name="sensor_namespace" value="$(arg sensor_namespace)" scope="global" />
+  <xacro:property name="pinger_namespace" value="$(arg pinger_namespace)" scope="global" />
+  <xacro:property name="namespace" value="$(arg namespace)" scope="global" />
   <!-- Include macros for dynamics plugins -->
   <xacro:include filename="$(find cora_description)/urdf/macros.xacro" />
+  <!-- Add a stereo camera pair -->
+  <xacro:wamv_camera name="front_left_camera"  y="0.1"  x="3.75" z="1.6" P="${radians(15)}" />
+  <xacro:wamv_camera name="front_right_camera" y="-0.1" x="3.75" z="1.6" P="${radians(15)}" />
+  <!-- Add simulated GPS -->
+  <xacro:wamv_gps name="gps" x="-0.4" z="1.4" />
+  <!-- Add Simulated IMU -->
+  <xacro:wamv_imu name="imu" y="-0.2" />
+  <!-- Add 3D LIDAR -->
+  <xacro:lidar name="front_lidar" type="16_beam" x="3.75" z="1.8" />
+  <!-- Add pinger -->
+  <xacro:wamv_pinger name="pinger" position="1.0 0 -1.0" />
   <!-- Attach hydrodynamics plugin -->
   <xacro:usv_dynamics_gazebo name="cora_dynamics_plugin" />

File: cora_description/urdf/macros.xacro (robot description, xacro)
@@ -3,4 +3,13 @@
 <robot xmlns:xacro="http://ros.org/wiki/xacro"
        name="cora">
+  <!-- Include sensor macros -->
+  <xacro:include filename="$(find wamv_gazebo)/urdf/sensors/wamv_camera.xacro" />
+  <xacro:include filename="$(find wamv_gazebo)/urdf/sensors/wamv_gps.xacro" />
+  <xacro:include filename="$(find wamv_gazebo)/urdf/sensors/wamv_imu.xacro" />
+  <xacro:include filename="$(find wamv_gazebo)/urdf/sensors/wamv_planar_lidar.xacro" />
+  <xacro:include filename="$(find wamv_gazebo)/urdf/sensors/wamv_3d_lidar.xacro" />
+  <xacro:include filename="$(find wamv_gazebo)/urdf/sensors/lidar.xacro" />
+  <xacro:include filename="$(find wamv_gazebo)/urdf/sensors/wamv_p3d.xacro" />
+  <xacro:include filename="$(find wamv_gazebo)/urdf/sensors/wamv_pinger.xacro" />
   <!-- Include dynamics macros -->
   <xacro:include filename="$(find wamv_gazebo)/urdf/dynamics/wamv_gazebo_dynamics_plugin.xacro" />

Commit message: first cut

File: cora_description/urdf/cora.urdf.xacro (robot description, xacro)
@@ -18,11 +18,9 @@
       </geometry>
     </collision>
-    <!-- Numbers are from MeshLab -->
+    <!-- Mass is calculated based on an estimate of draft, the effective length and the cross-section of
+a circle segment. The value for the draft is consistent specifications of similar vessels.  Moments of inertia are based on an effective cylindrical model-->
     <inertial>
-      <origin xyz="0.458797 0.002028 0.234834" rpy="0 0 0" />
-      <mass value="42.935"/>
-      <inertia ixx="55.373356" ixy="0.245103" ixz="-21.590300"
-                                iyy="341.188965" iyz="0.053122"
-                                                 izz="367.665375"/>
+       <mass value="33000.0"/>
+      <inertia ixx="20700.0" ixy="0.0" ixz="0.0" iyy="420000.0" iyz="0.0" izz="420000.0"/>
     </inertial>
   </link>

File: cora_description/urdf/macros.xacro (robot description, xacro)
@@ -4,4 +4,4 @@
        name="cora">
   <!-- Include dynamics macros -->
-  <xacro:include filename="$(find wamv_gazebo)/urdf/dynamics/wamv_gazebo_dynamics_plugin.xacro" />
+  <xacro:include filename="$(find cora_gazebo)/urdf/cora_gazebo_dynamics_plugin.xacro" />
 </robot>

Commit message: first tuning of dynamics and thrust

File: cora_description/urdf/cora.urdf.xacro (robot description, xacro)
@@ -6,7 +6,10 @@
     <parent link="base_link"/>
     <child link="dummy_link"/>
+    <!-- Adjust the visual/collision to match water height -->
+    <origin xyz="0 0 1" rpy="0 0 0"/>
   </joint>
   <link name="dummy_link">
     <visual>
+      <origin xyz="0 0 0" rpy="0 0 0" />
       <geometry>
         <mesh filename="package://cora_description/models/base/meshes/base.dae"/>

File: cora_description/urdf/thrusters.xacro (robot description, xacro)
@@ -23,5 +23,5 @@
   <joint name="left_chasis_engine_joint" type="revolute">
     <axis xyz="0 0 1"/>
-    <origin rpy="0 0 0" xyz="-6.103 0.911 -0.984"/>
+    <origin rpy="0 0 0" xyz="-6.103 0.911 0.016"/>
     <parent link="base_link"/>
     <child link="left_engine_link"/>
@@ -58,5 +58,5 @@
   <joint name="right_chasis_engine_joint" type="revolute">
     <axis xyz="0 0 1"/>
-    <origin rpy="0 0 0" xyz="-6.103 -0.911 -0.984"/>
+    <origin rpy="0 0 0" xyz="-6.103 -0.911 0.016"/>
     <parent link="base_link"/>
     <child link="right_engine_link"/>
@@ -75,8 +75,8 @@
       <cmdTimeout>1.0</cmdTimeout>
       <robotNamespace>${namespace}</robotNamespace>
-      <xacro:include filename="$(find wamv_gazebo)/urdf/thruster_layouts/wamv_gazebo_thruster_config.xacro" />
+      <xacro:include filename="$(find cora_gazebo)/urdf/cora_gazebo_thruster_config.xacro" />
       <!-- Angle must be disabled for VORC -->
-      <xacro:wamv_gazebo_thruster_config name="left" enable_angle="false" />
-      <xacro:wamv_gazebo_thruster_config name="right" enable_angle="false" />
+      <xacro:cora_gazebo_thruster_config name="left" />
+      <xacro:cora_gazebo_thruster_config name="right" />
     </plugin>
   </gazebo>

File: cora_gazebo/urdf/cora_gazebo_dynamics_plugin.xacro (robot description, xacro)
@@ -17,8 +17,8 @@
         <nDotR>0.0</nDotR>
         <!-- Linear and quadratic drag -->
-        <xU>0.0</xU>
-        <xUU>118.0</xUU>
-        <yV>0.0</yV>
-        <yVV>1345</yVV>
+        <xU>120.0</xU>
+        <xUU>240.0</xUU>
+        <yV>240.0</yV>
+        <yVV>2600</yVV>
         <zW>50000.0</zW>
 	<zWW>0.0</zWW>

Commit message: indentation
Signed-off-by: Mabel Zhang <mabel@openrobotics.org>

File: cora_description/urdf/cora.urdf.xacro (robot description, xacro)
@@ -25,5 +25,5 @@
     <inertial>
        <mass value="33000.0"/>
-      <inertia ixx="20700.0" ixy="0.0" ixz="0.0" iyy="420000.0" iyz="0.0" izz="420000.0"/>
+       <inertia ixx="20700.0" ixy="0.0" ixz="0.0" iyy="420000.0" iyz="0.0" izz="420000.0"/>
     </inertial>
   </link>

Commit message: cora model v.3 with textures; raised sensors z+=1
Signed-off-by: Mabel Zhang <mabel@openrobotics.org>

File: cora_description/urdf/cora.urdf.xacro (robot description, xacro)
@@ -13,6 +13,23 @@
       <origin xyz="0 0 0" rpy="0 0 0" />
       <geometry>
-        <mesh filename="package://cora_description/models/base/meshes/base.dae"/>
+        <mesh filename="package://cora_description/models/meshes/base.dae"/>
       </geometry>
+      <material name="base_material">
+        <diffuse>1.0 1.0 1.0</diffuse>
+        <specular>1.0 1.0 1.0</specular>
+        <pbr>
+          <metal>
+            <albedo_map>package://cora_description/models/materials/textures/Boat_Albedo.png</albedo_map>
+            <metalness_map>package://cora_description/models/materials/textures/Boat_Metalness.png</metalness_map>
+            <roughness_map>package://cora_description/models/materials/textures/Boat_Roughness.png</roughness_map>
+          </metal>
+        </pbr>
+        <!-- fallback to script if no PBR support-->
+        <script>
+          <uri>package://cora_description/models/materials/scripts/</uri>
+          <uri>package://cora_description/models/materials/textures/</uri>
+          <name>UrbanTile/Boat_Diffuse</name>
+        </script>
+      </material>
     </visual>
     <collision name="collision">

File: cora_description/urdf/cora.xacro (robot description, xacro)
@@ -22,9 +22,9 @@
   <xacro:property name="sensor_namespace" value="$(arg sensor_namespace)" scope="global" />
   <xacro:property name="pinger_namespace" value="$(arg pinger_namespace)" scope="global" />
-  <xacro:wamv_camera name="front_left_camera"  y="0.1"  x="3.75" z="1.6" P="${radians(15)}" />
-  <xacro:wamv_camera name="front_right_camera" y="-0.1" x="3.75" z="1.6" P="${radians(15)}" />
-  <xacro:lidar name="front_lidar" type="16_beam" x="3.75" z="1.8" />
-  <xacro:wamv_gps name="gps" x="-0.4" z="1.4" />
-  <xacro:wamv_imu name="imu" y="-0.2" />
+  <xacro:wamv_camera name="front_left_camera"  y="0.1"  x="3.75" z="2.6" P="${radians(15)}" />
+  <xacro:wamv_camera name="front_right_camera" y="-0.1" x="3.75" z="2.6" P="${radians(15)}" />
+  <xacro:lidar name="front_lidar" type="16_beam" x="3.75" z="2.8" />
+  <xacro:wamv_gps name="gps" x="-0.4" z="2.4" />
+  <xacro:wamv_imu name="imu" y="-0.2" z="1.0" />
   <xacro:wamv_pinger name="pinger" frameId="cora/pinger" />
 </robot>

File: cora_description/urdf/cora_v1.urdf.xacro (robot description, xacro)
@@ -10,5 +10,5 @@
     <visual>
       <geometry>
-        <mesh filename="package://cora_description/models/base/meshes/base_v1.dae"/>
+        <mesh filename="package://cora_description/models/meshes/base_v1.dae"/>
       </geometry>
     </visual>

File: cora_description/urdf/thrusters.xacro (robot description, xacro)
@@ -12,6 +12,23 @@
     <visual>
       <geometry>
-        <mesh filename="package://cora_description/models/propeller/meshes/propellerL.dae"/>
+        <mesh filename="package://cora_description/models/meshes/propellerL.dae"/>
       </geometry>
+      <material name="left_propeller_material">
+        <diffuse>1.0 1.0 1.0</diffuse>
+        <specular>1.0 1.0 1.0</specular>
+        <pbr>
+          <metal>
+            <albedo_map>package://cora_description/models/materials/textures/Boat_Albedo.png</albedo_map>
+            <metalness_map>package://cora_description/models/materials/textures/Boat_Metalness.png</metalness_map>
+            <roughness_map>package://cora_description/models/materials/textures/Boat_Roughness.png</roughness_map>
+          </metal>
+        </pbr>
+        <!-- fallback to script if no PBR support-->
+        <script>
+          <uri>package://cora_description/models/materials/scripts/</uri>
+          <uri>package://cora_description/models/materials/textures/</uri>
+          <name>UrbanTile/Boat_Diffuse</name>
+        </script>
+      </material>
     </visual>
     <inertial>
@@ -47,6 +64,23 @@
     <visual>
       <geometry>
-        <mesh filename="package://cora_description/models/propeller/meshes/propellerR.dae"/>
+        <mesh filename="package://cora_description/models/meshes/propellerR.dae"/>
       </geometry>
+      <material name="right_propeller_material">
+        <diffuse>1.0 1.0 1.0</diffuse>
+        <specular>1.0 1.0 1.0</specular>
+        <pbr>
+          <metal>
+            <albedo_map>package://cora_description/models/materials/textures/Boat_Albedo.png</albedo_map>
+            <metalness_map>package://cora_description/models/materials/textures/Boat_Metalness.png</metalness_map>
+            <roughness_map>package://cora_description/models/materials/textures/Boat_Roughness.png</roughness_map>
+          </metal>
+        </pbr>
+        <!-- fallback to script if no PBR support-->
+        <script>
+          <uri>package://cora_description/models/materials/scripts/</uri>
+          <uri>package://cora_description/models/materials/textures/</uri>
+          <name>UrbanTile/Boat_Diffuse</name>
+        </script>
+      </material>
     </visual>
     <inertial>

Commit message: Adding namespace for compatibility

File: cora_description/urdf/cora.urdf.xacro (robot description, xacro)
@@ -1,13 +1,13 @@
 <?xml version="1.0"?>
 <robot xmlns:xacro="http://ros.org/wiki/xacro" name="cora">
-  <link name="base_link">
+  <link name="cora/base_link">
   </link>
-  <joint name="dummy_joint" type="fixed">
-    <parent link="base_link"/>
-    <child link="dummy_link"/>
+  <joint name="cora/dummy_joint" type="fixed">
+    <parent link="cora/base_link"/>
+    <child link="cora/dummy_link"/>
     <!-- Adjust the visual/collision to match water height -->
     <origin xyz="0 0 1" rpy="0 0 0"/>
   </joint>
-  <link name="dummy_link">
+  <link name="cora/dummy_link">
     <visual>
       <origin xyz="0 0 0" rpy="0 0 0" />

File: cora_description/urdf/cora.xacro (robot description, xacro)
@@ -21,5 +21,5 @@
       <link name="cora_external_link"/>
       <joint name="cora_external_pivot_joint" type="universal">
-        <parent>cora::base_link</parent>
+        <parent>cora::cora/base_link</parent>
         <child>cora_external_link</child>
         <axis>
@@ -50,8 +50,12 @@
   <xacro:property name="sensor_namespace" value="$(arg sensor_namespace)" scope="global" />
   <xacro:property name="pinger_namespace" value="$(arg pinger_namespace)" scope="global" />
-  <xacro:wamv_camera name="front_left_camera"  x="-0.61" y="0.2"  z="4.7" post_z_from="4.6" P="${radians(15)}" />
-  <xacro:wamv_camera name="front_right_camera" x="-0.61" y="-0.2" z="4.7" post_z_from="4.6" P="${radians(15)}" />
-  <xacro:lidar name="front_lidar" type="16_beam" x="-0.595" z="5" P="${radians(8)}" post_z_from="4.6"/>
-  <xacro:wamv_gps name="gps" x="-1.0" z="4.6" lat="44.09525149" lon="9.823435727" update_rate="20" />
+  <xacro:wamv_camera name="front_left_camera"  x="-0.61" y="0.2"  z="4.7"
+  post_z_from="4.6" P="${radians(15)}" />
+  <xacro:wamv_camera name="front_right_camera" x="-0.61" y="-0.2" z="4.7"
+  post_z_from="4.6" P="${radians(15)}" />
+  <xacro:lidar name="front_lidar" type="16_beam" x="-0.595" z="5"
+  P="${radians(8)}" post_z_from="4.6"/>
+  <xacro:wamv_gps name="gps" x="-1.0" z="4.6"
+  	update_rate="20" />
   <xacro:wamv_imu name="imu" y="-0.2" z="1.0" update_rate="100" />
   <xacro:wamv_pinger name="pinger" frameId="cora/pinger" />

File: cora_description/urdf/cora_dynamics_plugin.xacro (robot description, xacro)
@@ -5,5 +5,5 @@
     <gazebo>
       <plugin name="usv_dynamics_${name}" filename="libusv_gazebo_dynamics_plugin.so">
-        <bodyName>base_link</bodyName>
+        <bodyName>cora/base_link</bodyName>
         <!-- Must be same as the ocean model!-->
         <waterLevel>0</waterLevel>

File: cora_description/urdf/thrusters.xacro (robot description, xacro)
@@ -41,5 +41,5 @@
     <axis xyz="0 0 1"/>
     <origin rpy="0 0 0" xyz="-6.103 0.911 0.016"/>
-    <parent link="base_link"/>
+    <parent link="cora/base_link"/>
     <child link="left_engine_link"/>
     <limit lower="${-pi}" upper="${pi}" effort="10" velocity="10"/>
@@ -93,5 +93,5 @@
     <axis xyz="0 0 1"/>
     <origin rpy="0 0 0" xyz="-6.103 -0.911 0.016"/>
-    <parent link="base_link"/>
+    <parent link="cora/base_link"/>
     <child link="right_engine_link"/>
     <limit lower="${-pi}" upper="${pi}" effort="10" velocity="10"/>
