Commit message: gymkhana scoring plugin
Signed-off-by: Mabel Zhang <mabel@openrobotics.org>

File: vorc_gazebo/worlds/gymkhana.world.xacro (robot description, xacro)
@@ -34,4 +34,79 @@
       <uri>model://obstacle_course</uri>
     </include>
+    <!-- Top-level scoring plugin -->
+    <plugin name="gymkhana_scoring_plugin"
+            filename="libgymkhana_scoring_plugin.so">
+      <vehicle>cora</vehicle>
+      <task_name>gymkhana</task_name>
+      <task_info_topic>/vorc/gymkhana/task/info</task_info_topic>
+      <contact_debug_topic>/vorc/gymkhana/debug/contact</contact_debug_topic>
+      <initial_state_duration>10</initial_state_duration>
+      <ready_state_duration>10</ready_state_duration>
+      <running_state_duration>300</running_state_duration>
+    </plugin>
+    <!-- Scoring plugin for buoy channel portion -->
+    <plugin name="navigation_scoring_plugin"
+            filename="libnavigation_scoring_plugin.so">
+      <vehicle>cora</vehicle>
+      <task_name>gymkhana_channel</task_name>
+      <task_info_topic>/vorc/gymkhana_channel/task/info</task_info_topic>
+      <contact_debug_topic>/vorc/gymkhana_channel/debug/contact</contact_debug_topic>
+      <initial_state_duration>10</initial_state_duration>
+      <ready_state_duration>10</ready_state_duration>
+      <running_state_duration>300</running_state_duration>
+      <collision_buffer>10</collision_buffer>
+      <release_joints>
+        <joint>
+          <name>cora_external_pivot_joint</name>
+        </joint>
+        <joint>
+          <name>cora_external_riser</name>
+        </joint>
+      </release_joints>
+      <course_name>short_navigation_course_0</course_name>
+      <obstacle_penalty>10.0</obstacle_penalty>
+      <gates>
+        <gate>
+          <left_marker>red_bound_0</left_marker>
+          <right_marker>green_bound_0</right_marker>
+        </gate>
+        <gate>
+          <left_marker>red_bound_1</left_marker>
+          <right_marker>green_bound_1</right_marker>
+        </gate>
+        <gate>
+          <left_marker>red_bound_2</left_marker>
+          <right_marker>green_bound_2</right_marker>
+        </gate>
+      </gates>
+    </plugin>
+    <!-- Scoring plugin for acoustic pinger portion -->
+    <plugin name="stationkeeping_scoring_plugin"
+          filename="libstationkeeping_scoring_plugin.so">
+      <vehicle>cora</vehicle>
+      <task_name>gymkhana_blackbox</task_name>
+      <rms_error_topic>/vorc/gymkhana_blackbox/rms_error</rms_error_topic>
+      <pose_error_topic>/vorc/gymkhana_blackbox/pose_error</pose_error_topic>
+      <goal_topic>/vorc/gymkhana_blackbox/goal</goal_topic>
+      <task_info_topic>/vorc/gymkhana_blackbox/task/info</task_info_topic>
+      <contact_debug_topic>/vorc/gymkhana_blackbox/debug/contact</contact_debug_topic>
+      <!-- Goal as Cartesian coordinates -->
+      <goal_pose_cart>116 -278 -5</goal_pose_cart>
+      <initial_state_duration>10</initial_state_duration>
+      <ready_state_duration>10</ready_state_duration>
+      <running_state_duration>300</running_state_duration>
+      <release_joints>
+        <joint>
+          <name>cora_external_pivot_joint</name>
+        </joint>
+        <joint>
+          <name>cora_external_riser</name>
+        </joint>
+      </release_joints>
+      <markers>
+        <scaling>0.2 0.2 2.0</scaling>
+        <height>0.5</height>
+      </markers>
+    </plugin>
   </world>
 </sdf>

File: vorc_gazebo/worlds/station_keeping.world.xacro (robot description, xacro)
@@ -20,5 +20,5 @@
       </wind_objs>
     </xacro:usv_wind_gazebo>
-  <plugin name="stationkeeping_scoring_plugin"
+    <plugin name="stationkeeping_scoring_plugin"
           filename="libstationkeeping_scoring_plugin.so">
       <vehicle>cora</vehicle>
